File: GRWatch.kicad_pcb (KiCad board)
At the start: 2 copper layers, 28 x 36 mm, 23 parts, among them J1 JST_SH_06, J2 JST_SH_04, SW1 SW_Push, SW2 SW_Push, SW3 SW_Push, U1 R5F100LJAFB, U2 BUZZER, U3 SSD1306, Y1 32.768k

Commit message: bug fix
Parts:
- added C10: 1.0uF, Capacitors_SMD:C_0805_HandSoldering, F.Cu at (105.2, 113.3)
- added C11: 0.1uF, Capacitors_SMD:C_0805_HandSoldering, F.Cu at (110.2, 113.3)
- added C9: 1.0uF, Capacitors_SMD:C_0805_HandSoldering, F.Cu at (102.9, 113.3)
- added R5: 10k, Resistors_SMD:R_0805_HandSoldering, F.Cu at (115.3, 113.3)
- added R6: 10k, Resistors_SMD:R_0805_HandSoldering, F.Cu at (112.8, 113.3)
- added R7: 10k, Resistors_SMD:R_0805_HandSoldering, F.Cu at (107.7, 113.3)
- C7: value 2.2uF -> 4.7uF
- G***: moved to B.Cu
- R4: value 400k -> 390k
- SW1, SW2, SW3: footprint misc:THAM16 -> misc:SKSC
- moved G*** 3.53 mm to (113.0, 112.0), turned to 180 degrees
- moved SW2 0.82 mm to (121.5, 93.0)
- moved SW1 0.80 mm to (121.5, 102.7)
- moved SW3 0.80 mm to (121.5, 112.2)
Connections:
- J1 pad M1: (no net) -> Net-(J1-PadM1)
- J1 pad M2: (no net) -> Net-(J1-PadM2)
- J2 pad M1: (no net) -> Net-(J2-PadM1)
- J2 pad M2: (no net) -> Net-(J2-PadM2)
- U1 pad 1: (no net) -> Net-(U1-Pad1)
- U1 pad 19: (no net) -> Net-(U1-Pad19)
- U1 pad 2: (no net) -> Net-(U1-Pad2)
- U1 pad 20: (no net) -> Net-(U1-Pad20)
- U1 pad 22: (no net) -> Net-(U1-Pad22)
- U1 pad 23: (no net) -> Net-(U1-Pad23)
- U1 pad 24: (no net) -> Net-(U1-Pad24)
- U1 pad 25: (no net) -> Net-(U1-Pad25)
- U1 pad 26: (no net) -> Net-(U1-Pad26)
- U1 pad 27: (no net) -> Net-(U1-Pad27)
- U1 pad 28: (no net) -> Net-(U1-Pad28)
- U1 pad 29: (no net) -> Net-(U1-Pad29)
- U1 pad 3: (no net) -> Net-(U1-Pad3)
- U1 pad 30: (no net) -> Net-(U1-Pad30)
- U1 pad 31: (no net) -> Net-(U1-Pad31)
- U1 pad 33: (no net) -> Net-(U1-Pad33)
- U1 pad 34: (no net) -> Net-(U1-Pad34)
- U1 pad 35: (no net) -> Net-(U1-Pad35)
- U1 pad 36: (no net) -> Net-(U1-Pad36)
- U1 pad 37: (no net) -> Net-(U1-Pad37)
- U1 pad 38: (no net) -> Net-(U1-Pad38)
- U1 pad 39: (no net) -> Net-(U1-Pad39)
- U1 pad 4: (no net) -> Net-(U1-Pad4)
- U1 pad 41: (no net) -> Net-(U1-Pad41)
- U1 pad 43: (no net) -> Net-(U1-Pad43)
- U1 pad 46: (no net) -> Net-(U1-Pad46)
- U1 pad 47: (no net) -> Net-(U1-Pad47)
- U1 pad 48: (no net) -> Net-(U1-Pad48)
- U1 pad 49: (no net) -> Net-(U1-Pad49)
- U1 pad 50: (no net) -> Net-(U1-Pad50)
- U1 pad 51: (no net) -> Net-(U1-Pad51)
- U1 pad 52: (no net) -> Net-(U1-Pad52)
- U1 pad 57: (no net) -> Net-(U1-Pad57)
- U1 pad 58: (no net) -> Net-(U1-Pad58)
- U1 pad 61: (no net) -> Net-(U1-Pad61)
- U1 pad 62: (no net) -> Net-(U1-Pad62)
- U1 pad 63: (no net) -> Net-(U1-Pad63)
- U1 pad 64: (no net) -> Net-(U1-Pad64)
- U2 pad 3: (no net) -> Net-(U2-Pad3)
- U2 pad 4: (no net) -> Net-(U2-Pad4)
- U3 pad 1: (no net) -> GND
- U3 pad 11: +3V3 -> Net-(C11-Pad1)
- U3 pad 14: +3V3 -> Net-(C11-Pad1)
- U3 pad 30: (no net) -> GND
- U3 pad 7: (no net) -> Net-(U3-Pad7)
Routing:
- net GND: track 170.1 -> 196.8 mm
- net Net-(C11-Pad1): track 0.00 -> 16.1 mm
- net +3V3: track 108.5 -> 120.8 mm
- net SDA: track 7.26 -> 13.6 mm
- net SCL: track 6.33 -> 12.2 mm
- net SW3: track 14.8 -> 19.6 mm
- net SW1: track 6.04 -> 7.46 mm
- net SW2: track 7.27 -> 8.63 mm
- net Net-(C6-Pad2): track 9.38 -> 8.87 mm
Other:
- outline, holes or cut-outs redrawn
