File: GRWatch.sch (KiCad schematic (older format))
At the start: 19 parts, among them J1 JST_SH_06, U1 R5F100LJAFB, U2 MULTI_SW, U3 SSD1306, U5 BUZZER, Y1 32.768k

Commit message: add tiny version
Parts:
- removed U2: MULTI_SW, misc:TST-1005, symbol MULTI_SW
- removed U5: BUZZER, misc:BZ7025, symbol BUZZER
- added J2: JST_SH_04, JST-SH:JST-SM-04B-SRSS-TB, symbol JST_SH_04
- added SW1, SW2, SW3: SW_Push, misc:THAM16, symbol SW_Push
- added U2: BUZZER, misc:BZ7025_3pin, symbol BUZZER
Connections:
- net GND: now also SW1.2, SW2.2, SW3.2, U2.2 (-)
- net SW1: now also SW1.1
- net SW2: now also SW2.1
- net SW3: now also SW3.1
- net at U1.42 (P14/RxD2/SI20/SDA20/(SCLA0)/(TI03)/(TO03)): now also U2.1 (+)
- net A1: now reaches U1.53 (P23/ANI3)
- net A1: now also J2.1 (P1)
- net A0: now reaches U1.54 (P22/ANI2)
- net A0: now also J2.2 (P2)
- net D8: now reaches U1.59 (P03/ANI16/SI10/RxD1/SDA10)
- net D8: now also J2.3 (P3)
- net D7: now reaches U1.60 (P02/ANI17/SO10/TxD1)
- net D7: now also J2.4 (P4)
- no-connect marks 46 -> 44

Commit message: bug fix
Parts:
- added C10, C9: 1.0uF, Capacitors_SMD:C_0805_HandSoldering, symbol C
- added C11: 0.1uF, Capacitors_SMD:C_0805_HandSoldering, symbol C
- added R5, R6, R7: 10k, Resistors_SMD:R_0805_HandSoldering, symbol R
- C7: value 2.2uF -> 4.7uF
- R4: value 400k -> 390k
- SW1, SW2, SW3: footprint misc:THAM16 -> misc:SKSC
Connections:
- net +3V3: now also C10.1, C9.1, R5.1, R6.1, R7.2; no longer U3.11 (BS1), U3.14 (/RES)
- net GND: now also U3.1 (NC(GND)), U3.30 (NC(GND)), C10.2, C11.2, C9.2
- net SCL: now also R6.2
- net SDA: now also R5.2
- new net: C11.1, R7.1, U3.11 (BS1), U3.14 (/RES)
- no-connect marks 44 -> 42
Other:
- moved on the sheet: C7
